File: PCB/macropad.kicad_pcb (KiCad board)
At the start: 2 copper layers, 60 x 70.2 mm, 46 parts, among them J1 USB_C_Receptacle_USB2.0_16P, SW1 SW_Push, SW2 SW_Push, SW3 SW_Push, SW4 SW_Push, SW5 SW_Push, SW6 SW_Push, SW7 SW_Push, SW8 SW_Push, SW9 SW_Push, U1 ESP32-C6-MINI-1, U2 AZ1117CH2-3.3

Commit message: Update macropad.kicad_pcb
Parts:
- added G***: LOGO, LOGO, B.Cu at (113.3, 82.2)
